Commit message: poprawiony dh_to_rpy, skonczone modele sztywne i ruchome

File: lab2/urdf/model.xacro (robot description, xacro)
@@ -1,5 +1,9 @@
 <?xml version="1.0"?>
 <robot name="PatoBombelDaughter" xmlns:xacro="http://ros.org/wiki/xacro">
-	<xacro:property name="pi" value="3.1415" />
+	<!-- Wartości parametrow -->
+	<xacro:property name="a2" value="0.3" />
+	<xacro:property name="base_size" value="0.25" />
+	<xacro:property name="gripper_size" value="0.2" />
+	<!-- Stworzenie kolorow pokryc elementow -->
 	<material name="blue">
 		<color rgba="0 0 0.8 1"/>
@@ -11,5 +15,6 @@
 		<color rgba="1 1 1 1"/>
 	</material>
-	<xacro:macro name="segmentMacro" params="name rpy xyz size">
+	<!-- Makro segmentMacro tworzace link - element robota -->
+	<xacro:macro name="segmentMacro" params="name color xyz size">
 		<link name="${name}">
 			<visual>
@@ -17,22 +22,25 @@
 					<box size="${size}"/>
 				</geometry>
-				<material name="blue"/>
-				<origin rpy="${rpy}" xyz="${xyz}"/>
+				<material name="${color}"/>
+				<origin xyz="${xyz}"/>
 			</visual>
 		</link>
 	</xacro:macro>
-	<xacro:macro name="jointFixed" params="parent child origin_xyz">
+	<!-- Makro jointFixed tworzące joint - tworzace sztywne polaczenie pomiedzy elementami robota -->
+	<xacro:macro name="jointFixed" params="parent child rpy xyz">
 		<joint name="${parent}_to_${child}_joint_fixed" type="fixed">
 			<parent link="${parent}"/>
 			<child link="${child}"/>
-			<origin xyz="${origin_xyz}"/>
+			<origin rpy="${rpy}" xyz="${xyz}"/>
 		</joint>
 	</xacro:macro>
-	<xacro:segmentMacro name="base"      rpy="0 0 0" xyz="0 0 0.1"          size="0.2 0.2 0.2"/>
-	<xacro:segmentMacro name="segment_1" rpy="0 0 0" xyz="0 0 ${0.45+0.01}" size="0.1 0.1 0.5"/>
-	<xacro:segmentMacro name="segment_2" rpy="0 0 0" xyz="0 0 ${0.95+0.02}" size="0.1 0.1 0.5"/>
-	<xacro:segmentMacro name="gripper"   rpy="0 0 0" xyz="0 0 ${1.25+0.03}" size="0.1 0.1 0.1"/>
-	<xacro:jointFixed parent="base"      child="segment_1" origin_xyz="0 0 0.2" />
-	<xacro:jointFixed parent="segment_1" child="segment_2" origin_xyz="0 0 0.90"/>
-	<xacro:jointFixed parent="segment_2" child="gripper"   origin_xyz="0 0 1.0" />
+	<!-- Wykorzystanie makra segmentMacro do stworzenia elementow robota -->
+	<xacro:segmentMacro name="base_link" color="black" xyz="0 0 ${base_size/2}"     size="0.2 0.2 ${base_size}"/>
+	<xacro:segmentMacro name="segment_1" color="white" xyz="0 0 ${0}"               size="0 0 0"/>
+	<xacro:segmentMacro name="segment_2" color="blue"  xyz="${a2/2} 0 0 "           size="${a2} 0.1 0.1 "/>
+	<xacro:segmentMacro name="gripper"   color="white" xyz="${gripper_size/2} 0 0 " size="${gripper_size} 0.1 0.1 "/>
+	<!-- Wykorzystanie makra jointFixed do stworzenia polaczen pomiedzy elementami robota -->
+	<xacro:jointFixed parent="base_link" child="segment_1" rpy="0 0 0"        xyz="0 0 ${base_size}" />
+	<xacro:jointFixed parent="segment_1" child="segment_2" rpy="${-pi/2} 0 0" xyz="0 0 0"            />
+	<xacro:jointFixed parent="segment_2" child="gripper"   rpy="0 0 0"        xyz="${a2} 0 0"        />
 </robot>

File: lab2/urdf/modelMovable.xacro (robot description, xacro)
@@ -1,5 +1,9 @@
 <?xml version="1.0"?>
 <robot name="PatoBombelSon" xmlns:xacro="http://ros.org/wiki/xacro">
-	<xacro:property name="pi" value="3.1415" />
+	<!-- Wartości parametrow -->
+	<xacro:property name="a2" value="0.3" />
+	<xacro:property name="base_size" value="0.25" />
+	<xacro:property name="gripper_size" value="0.2" />
+	<!-- Stworzenie kolorow pokryc elementow -->
 	<material name="blue">
 		<color rgba="0 0 0.8 1"/>
@@ -11,5 +15,6 @@
 		<color rgba="1 1 1 1"/>
 	</material>
-	<xacro:macro name="segmentMacro" params="name rpy xyz size">
+	<!-- Makro segmentMacro tworzace link - element robota -->
+	<xacro:macro name="segmentMacro" params="name color xyz size">
 		<link name="${name}">
 			<visual>
@@ -17,24 +22,30 @@
 					<box size="${size}"/>
 				</geometry>
-				<material name="blue"/>
-				<origin rpy="${rpy}" xyz="${xyz}"/>
+				<material name="${color}"/>
+				<origin xyz="${xyz}"/>
 			</visual>
 		</link>
 	</xacro:macro>
-	<xacro:macro name="jointContinuous" params="parent child origin_xyz axis_rpy axis_xyz">
-		<joint name="${parent}_to_${child}_joint_continuous" type="continuous">
-			<limit effort="1000.0" lower="0.0" upper="1.0" velocity="0.5"/>
-			<axis rpy="${axis_rpy}" xyz="${axis_xyz}"/>
+	<!-- Makro jointRevolute tworzące joint - tworzace ruchome polaczenie pomiedzy elementami robota -->
+	<xacro:macro name="jointRevolute" params="parent child rpy xyz  axis_xyz limit_low limit_up">
+		<joint name="${parent}_to_${child}_joint_continuous" type="revolute">
+			<limit effort="1000.0" lower="${limit_low}" upper="${limit_up}" velocity="0.5"/>
+			<axis  xyz="${axis_xyz}"/>
 			<parent link="${parent}"/>
 			<child link="${child}"/>
-			<origin xyz="${origin_xyz}"/>
+			<origin rpy="${rpy}" xyz="${xyz}"/>
 		</joint>
 	</xacro:macro>
-	<xacro:segmentMacro name="base"      rpy="0 0 0" xyz="0 0 0.1"          size="0.2 0.2 0.2"/>
-	<xacro:segmentMacro name="segment_1" rpy="0 0 0" xyz="0 0 ${0.45+0.01}" size="0.1 0.1 0.5"/>
-	<xacro:segmentMacro name="segment_2" rpy="0 0 0" xyz="0 0 ${0.95+0.02}" size="0.1 0.1 0.5"/>
-	<xacro:segmentMacro name="gripper"   rpy="0 0 0" xyz="0 0 ${1.25+0.03}" size="0.1 0.1 0.1"/>
-	<xacro:jointContinuous parent="base"      child="segment_1" origin_xyz="0 0 0.2"  axis_rpy="0 0 1" axis_xyz="0 0 0.2"/>
-	<xacro:jointContinuous parent="segment_1" child="segment_2" origin_xyz="0 0 0.90" axis_rpy="0 1 0" axis_xyz="0 0 1.1"/>
-	<xacro:jointContinuous parent="segment_2" child="gripper"   origin_xyz="0 0 1.5"  axis_rpy="1 0 0" axis_xyz="0 0 1.9"/>
+	<!-- Wykorzystanie makra segmentMacro do stworzenia elementow robota -->
+	<xacro:segmentMacro name="base_link" color="black" xyz="0 0 ${base_size/2}"     size="0.2 0.2 ${base_size}"/>
+	<xacro:segmentMacro name="segment_1" color="white" xyz="0 0 ${0}"               size="0 0 0"/>
+	<xacro:segmentMacro name="segment_2" color="blue"  xyz="${a2/2} 0 0 "           size="${a2} 0.1 0.1 "/>
+	<xacro:segmentMacro name="gripper"   color="white" xyz="${gripper_size/2} 0 0 " size="${gripper_size} 0.1 0.1 "/>
+	<!-- Wykorzystanie makra jointRevolute do stworzenia polaczen pomiedzy elementami robota -->
+	<xacro:jointRevolute parent="base_link" child="segment_1" rpy="0 0 0"        xyz="0 0 ${base_size}"
+		axis_xyz="0 0 1" limit_low="-3.14" limit_up="3.14"/>
+	<xacro:jointRevolute parent="segment_1" child="segment_2" rpy="${-pi/2} 0 0" xyz="0 0 0"
+		axis_xyz="0 0 1" limit_low="-1.54" limit_up="0"/>
+	<xacro:jointRevolute parent="segment_2" child="gripper"   rpy="0 0 0"        xyz="${a2} 0 0"
+		axis_xyz="0 0 1" limit_low="0" limit_up="1.54"/>
 </robot>
