Commit message: uwzglednienie wysokosci bazy w nondkl, nonkdl nadal publikuje tylko position

File: lab3/urdf/modelMovable.xacro (robot description, xacro)
@@ -2,7 +2,7 @@
 <robot name="PatoBombelSon" xmlns:xacro="http://ros.org/wiki/xacro">
 	<!-- Wartości parametrow -->
-	<xacro:property name="a2" value="0.3" />
-	<xacro:property name="base_size" value="0.25" />
-	<xacro:property name="gripper_size" value="0.2" />
+	<xacro:property name="a2" value="0.5" />
+	<xacro:property name="base_size" value="0.2" />
+	<xacro:property name="gripper_size" value="0.01" />
 	<!-- Stworzenie kolorow pokryc elementow -->
 	<material name="blue">

Commit message: Ostatnie poprawki na laboratorium

File: lab3/urdf/modelMovable.xacro (robot description, xacro)
@@ -2,7 +2,7 @@
 <robot name="PatoBombelSon" xmlns:xacro="http://ros.org/wiki/xacro">
 	<!-- Wartości parametrow -->
-	<xacro:property name="a2" value="0.5" />
-	<xacro:property name="base_size" value="0.2" />
-	<xacro:property name="gripper_size" value="0.01" />
+	<xacro:property name="a2" value="$(arg a2)" />
+	<xacro:property name="base_size" value="$(arg base_size)" />
+	<xacro:property name="gripper_size" value="$(arg gripper_size)" />
 	<!-- Stworzenie kolorow pokryc elementow -->
 	<material name="blue">
