Commit message: modelMovable-dodane narzedzie jako dodatkowy link, config.rviz-dopasowanie do zmian modelu

File: lab4/urdf/modelMovable.xacro (robot description, xacro)
@@ -42,4 +42,5 @@
 	<xacro:segmentMacro name="segment_2" color="blue"  xyz="${a2/2} 0 0 "           size="${a2} 0.1 0.1 "/>
 	<xacro:segmentMacro name="gripper"   color="white" xyz="${gripper_size/2} 0 0 " size="${gripper_size} 0.1 0.1 "/>
+	<xacro:segmentMacro name="gripperTool"   color="black" xyz="0 0 0 " size="0 0.1 0.1 "/>
 	<!-- Wykorzystanie makra jointRevolute do stworzenia polaczen pomiedzy elementami robota -->
 	<xacro:jointRevolute parent="base_link" child="segment_1" rpy="0 0 0"        xyz="0 0 ${base_size}"
@@ -49,3 +50,8 @@
 	<xacro:jointRevolute parent="segment_2" child="gripper"   rpy="0 0 0"        xyz="${a2} 0 0"
 		axis_xyz="0 0 1" limit_low="0" limit_up="1.54"/>
+	<joint name="gripperTool_to_gripper_joint_continuous" type="fixed">
+		<parent link="gripper"/>
+		<child link="gripperTool"/>
+		<origin rpy="0 0 0" xyz="${gripper_size} 0 0"/>
+	</joint>
 </robot>
